File: fcch-laser-controller.kicad_pcb (KiCad board)
At the start: 2 copper layers, 90 x 80 mm, 31 parts, among them J1 Barrel_Jack_Switch, J10 Conn_01x03_Male, J11 Conn_01x02_Male, J12 Conn_01x04_Male, J13 Conn_01x19_Male, J14 Conn_01x19_Male, J2 Barrel_Jack_Switch, J3 Barrel_Jack_Switch, J4 Barrel_Jack_Switch, J5 Conn_02x03_Odd_Even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

Commit message: pcb: use commas for labels
This takes up less space, leaving slightly larger gaps between the labels
for adjacent connectors.
Other:
- board text added: "5V,3V3,AIR,GND"
- board text added: "FCCH Laser Controller v1a 2022/01/28 Stephen Warren"
- board text added: "PWM,GND"
- board text added: "STP,DIR,EN GND,GND,GND"
- board text added: "V24,LIM,GND"
- board text removed: "5V 3V3 AIR GND"
- board text removed: "FCCH Laser Controller v1 2022/01/25 Stephen Warren"
- board text removed: "PWM GND"
- board text removed: "STP DIR EN GND GND GND"
- board text removed: "V24 LIM GND"
Changed lines of the file:
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@@
     (effects (font (size 1 1) (thickness 0.15)))
   )
-  (gr_text "STP DIR  EN\nGND GND GND" (at 144.78 147.32) (layer F.SilkS)
+  (gr_text "STP,DIR,EN\nGND,GND,GND" (at 144.78 147.32) (layer F.SilkS)
     (effects (font (size 1 1) (thickness 0.15)))
   )
-  (gr_text "STP DIR  EN\nGND GND GND" (at 158.75 147.32) (layer F.SilkS)
+  (gr_text "STP,DIR,EN\nGND,GND,GND" (at 158.75 147.32) (layer F.SilkS)
     (effects (font (size 1 1) (thickness 0.15)))
   )
@@
     (effects (font (size 1.5 1) (thickness 0.15)))
   )
-  (gr_text "FCCH Laser Controller\nv1 2022/01/25\nStephen Warren" (at 123.19 146.05) (layer F.SilkS)
+  (gr_text "FCCH Laser Controller\nv1a 2022/01/28\nStephen Warren" (at 123.19 146.05) (layer F.SilkS)
     (effects (font (size 1 1) (thickness 0.125)))
   )
@@
     (effects (font (size 1.5 1) (thickness 0.15)))
   )
-  (gr_text "PWM GND" (at 100.965 92.71 90) (layer F.SilkS)
+  (gr_text PWM,GND (at 100.965 92.71 90) (layer F.SilkS)
     (effects (font (size 1 1) (thickness 0.15)))
   )
-  (gr_text "5V 3V3 AIR GND" (at 100.965 102.87 90) (layer F.SilkS)
+  (gr_text 5V,3V3,AIR,GND (at 100.965 102.87 90) (layer F.SilkS)
     (effects (font (size 1 1) (thickness 0.15)))
   )
-  (gr_text "V24 LIM GND" (at 100.965 114.3 90) (layer F.SilkS)
+  (gr_text V24,LIM,GND (at 100.965 114.3 90) (layer F.SilkS)
     (effects (font (size 1 1) (thickness 0.15)))
   )
-  (gr_text "V24 LIM GND" (at 100.965 134.62 90) (layer F.SilkS)
+  (gr_text V24,LIM,GND (at 100.965 134.62 90) (layer F.SilkS)
     (effects (font (size 1 1) (thickness 0.15)))
   )
@@
   (gr_circle (center 106.68 128.27) (end 106.93 128.27) (layer F.SilkS) (width 0.5))
   (gr_circle (center 106.68 138.43) (end 106.93 138.43) (layer F.SilkS) (width 0.5))
-  (gr_text "V24 LIM GND" (at 100.965 124.46 90) (layer F.SilkS)
+  (gr_text V24,LIM,GND (at 100.965 124.46 90) (layer F.SilkS)
     (effects (font (size 1 1) (thickness 0.15)))
   )
-  (gr_text "STP DIR  EN\nGND GND GND" (at 172.72 147.32) (layer F.SilkS)
+  (gr_text "STP,DIR,EN\nGND,GND,GND" (at 172.72 147.32) (layer F.SilkS)
     (effects (font (size 1 1) (thickness 0.15)))
   )
